File: AP63203 1x1/SparkFun Buck Regulator Breakout - AP63203.brd (EAGLE design)
At the start: 25.4 x 25.4 mm, 38 parts, among them U1 AP63203

Commit message: v01 update
-Added barrel jack
-Replaced 4.7uF capacitors with 10uF/50V
Parts:
- removed C5: 22uF, SparkFun-Capacitors:0603
- added J3: POWER_JACK, SparkFun-Connectors:POWER_JACK_PTH_SLOT
- added U$17: (no value), SparkFun-Aesthetics:SFE_LOGO_FLAME_.1
- C1: value 4.7uF -> 10uF; device SparkFun-Capacitors:0603 -> SparkFun-Capacitors:1210
- C2: value 4.7uF -> 0.1uF
- C3: value 0.1uF -> 22uF
- FD2: value FIDUCIAL0.2MM -> FIDUCIALUFIDUCIAL; device SparkFun-Aesthetics:FIDUCIAL-0.2MM -> SparkFun-Aesthetics:FIDUCIAL-MICRO
- U$8: device output:#3V8_#_32V#0 -> output:#VIN#0
- moved LOGO1 19.0 mm to (12.7, 21.0), flipped to the bottom
- moved LOGO2 7.62 mm to (12.7, 14.0)
- moved C2 6.78 mm to (10.9, 18.5)
- moved C3 5.51 mm to (14.4, 12.3), turned to 180 degrees
- moved R2 3.64 mm to (11.2, 10.5), turned to 180 degrees
- moved C4 3.43 mm to (14.4, 13.8)
- moved C1 2.71 mm to (8.89, 13.1)
- moved R1 2.25 mm to (7.87, 10.5)
- moved U1 1.91 mm to (9.78, 16.1)
- moved L1 1.90 mm to (15.0, 16.9)
- moved U$15 1.78 mm to (10.9, 23.4)
Connections:
- net 3.3V: now also C3.1; no longer C5.1
- net GND: now also C3.2, J3.GND; no longer C2.2, C5.2
- net N$4: now also C2.1; no longer C3.1
- net N$5: now also C2.2; no longer C3.2
- net VIN: now also J3.PWR; no longer C2.1
Routing:
- net VIN: track 22.0 -> 17.4 mm
- net EN: track 18.3 -> 21.2 mm

Commit message: v01 post view changes
Parts:
- added D1: RED, SparkFun-LED:LED-0603
- added LOGO3: SPECIAL_INSTRUCTIONS-ORDERING, SparkFun-Aesthetics:ORDERING_INSTRUCTIONS
- added PWR: (no value), SparkFun-Jumpers:SMT-JUMPER_2_NC_TRACE_SILK
- added R3: 1k, SparkFun-Resistors:0603
- added U$18: (no value), buzzard_labels (1):PWR1
- added U$19: (no value), buzzard_labels (3):PWR1
- LOGO2: value OSHW-LOGOM -> OSHW-LOGOS; device SparkFun-Aesthetics:OSHW-LOGO-M -> SparkFun-Aesthetics:OSHW-LOGO-S
- moved LOGO2 9.78 mm to (12.7, 4.19)
- moved C2 1.65 mm to (9.27, 18.5)
- moved U1 1.65 mm to (8.13, 16.1)
- moved L1 1.27 mm to (13.7, 16.9)
- moved C3 0.64 mm to (13.7, 12.3)
- moved C4 0.64 mm to (13.7, 13.8)
- moved C1 0.25 mm to (8.64, 13.1)
- moved R1 0.25 mm to (7.62, 10.5)
- moved R2 0.25 mm to (10.9, 10.5)
Connections:
- new net N$1: D1.A, R3.1
- new net N$2: PWR.1, R3.2
- net 3.3V: now also PWR.2
- net GND: now also D1.C
Routing:
- net N$2: track 0.00 -> 2.81 mm, vias 0 -> 1
- net 3.3V: track 0.25 -> 2.51 mm, vias 0 -> 1
- net N$1: track 0.00 -> 1.81 mm
- net EN: track 21.2 -> 20.6 mm
Other:
- board text added: "2oz copper"
