File: AP63203 Small/SparkFun Buck Regulator Breakout - AP63203.sch (EAGLE design)
At the start: 17 parts, among them U1 AP63203

Commit message: v01 post view changes
Parts:
- removed C5: 22uF, SparkFun-Capacitors:22UF-0603-6.3V-20%
- added LOGO3: SPECIAL_INSTRUCTIONS-ORDERING, SparkFun-Aesthetics:SPECIAL_INSTRUCTIONS-ORDERING
- C1: value 4.7uF -> 10uF; device SparkFun-Capacitors:4.7UF-0603-35V-(20%) -> SparkFun-Capacitors:10UF-1210-50V-20%
- C2: value 4.7uF -> 0.1uF; device SparkFun-Capacitors:4.7UF-0603-35V-(20%) -> SparkFun-Capacitors:0.1UF-0603-25V-5%
- C3: value 0.1uF -> 22uF; device SparkFun-Capacitors:0.1UF-0603-25V-5% -> SparkFun-Capacitors:22UF-0603-6.3V-20%
Connections:
- net 3.3V: now also C3.1; no longer C5.1
- net GND: now also C3.2; no longer C2.2, C5.2
- net N$4: now also C2.1; no longer C3.1
- net N$5: now also C2.2; no longer C3.2
- net VIN: no longer C2.1
Other:
- note added: "Buck Regulator"
- note added: "Connector"
- note added: "VIN: 3.8 - 32V Iout: 2A Max"
- moved on the sheet: C1, C2, C3, C4, L1, R1, R2, U1
