File: AP63203 Small/SparkFun Buck Regulator Breakout - AP63203.brd (EAGLE design)
At the start: 12.7 x 10.2 mm, 24 parts, among them U1 AP63203

Commit message: v01 post view changes
Parts:
- removed C5: 22uF, SparkFun-Capacitors:0603
- added LOGO3: SPECIAL_INSTRUCTIONS-ORDERING, SparkFun-Aesthetics:ORDERING_INSTRUCTIONS
- C1: value 4.7uF -> 10uF; device SparkFun-Capacitors:0603 -> SparkFun-Capacitors:1210
- C2: value 4.7uF -> 0.1uF
- C3: value 0.1uF -> 22uF
- moved C3 7.11 mm to (9.27, 2.79), turned to 180 degrees
- moved C2 4.94 mm to (5.84, 9.02)
- moved C4 1.52 mm to (9.27, 4.32)
- moved C1 1.09 mm to (4.95, 3.68)
Connections:
- net 3.3V: now also C3.1; no longer C5.1
- net GND: now also C3.2; no longer C2.2, C5.2
- net N$4: now also C2.1; no longer C3.1
- net N$5: now also C2.2; no longer C3.2
- net VIN: no longer C2.1
Other:
- board text added: "2oz copper"
Changed lines of the file:
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@@
 <?xml version="1.0" encoding="utf-8"?>
 <!DOCTYPE eagle SYSTEM "eagle.dtd">
-<eagle version="9.5.2">
+<eagle version="9.6.2">
 <drawing>
 <settings>
@@
 <layer number="37" name="tTest" color="7" fill="1" visible="no" active="yes"/>
 <layer number="38" name="bTest" color="7" fill="1" visible="no" active="yes"/>
-<layer number="39" name="tKeepout" color="4" fill="11" visible="no" active="yes"/>
-<layer number="40" name="bKeepout" color="1" fill="11" visible="no" active="yes"/>
+<layer number="39" name="tKeepout" color="4" fill="11" visible="yes" active="yes"/>
+<layer number="40" name="bKeepout" color="1" fill="11" visible="yes" active="yes"/>
 <layer number="41" name="tRestrict" color="4" fill="10" visible="no" active="yes"/>
 <layer number="42" name="bRestrict" color="1" fill="10" visible="no" active="yes"/>
@@
 <layer number="45" name="Holes" color="7" fill="1" visible="yes" active="yes"/>
 <layer number="46" name="Milling" color="3" fill="1" visible="no" active="yes"/>
-<layer number="47" name="Measures" color="7" fill="1" visible="yes" active="yes"/>
+<layer number="47" name="Measures" color="7" fill="1" visible="no" active="yes"/>
 <layer number="48" name="Document" color="7" fill="1" visible="no" active="yes"/>
 <layer number="49" name="Reference" color="7" fill="1" visible="no" active="yes"/>
@@
 <text x="10.16" y="-15.24" size="1.778" layer="51" font="vector" ratio="15">Alex Wende</text>
 <text x="12.192" y="9.779" size="1.016" layer="16" font="vector" ratio="15" rot="SMR270">v01</text>
+<text x="25.4" y="31.75" size="1.778" layer="51" font="vector" ratio="15">2oz copper</text>
 </plain>
 <attributes>
@@
 </autorouter>
 <elements>
-<element name="C3" library="SparkFun-Capacitors" package="0603" value="0.1uF" x="5.842" y="9.017" smashed="yes">
+<element name="C2" library="SparkFun-Capacitors" package="0603" value="0.1uF" x="5.842" y="9.017" smashed="yes">
 <attribute name="NAME" x="5.842" y="9.779" size="0.6096" layer="25" font="vector" ratio="20" align="bottom-center"/>
 <attribute name="PROD_ID" value="CAP-08604" x="37.592" y="-2.413" size="1.778" layer="27" display="off"/>
 <attribute name="VALUE" x="5.842" y="8.255" size="0.6096" layer="27" font="vector" ratio="20" align="top-center"/>
 </element>
-<element name="C4" library="SparkFun-Capacitors" package="0603" value="22uF" x="9.271" y="2.794" smashed="yes" rot="R180">
+<element name="C3" library="SparkFun-Capacitors" package="0603" value="22uF" x="9.271" y="2.794" smashed="yes" rot="R180">
 <attribute name="NAME" x="9.271" y="2.032" size="0.6096" layer="25" font="vector" ratio="20" rot="R180" align="bottom-center"/>
 <attribute name="PROD_ID" value="CAP-14464" x="-26.289" y="14.224" size="1.778" layer="27" rot="R180" display="off"/>
 <attribute name="VALUE" x="9.271" y="3.556" size="0.6096" layer="27" font="vector" ratio="20" rot="R180" align="top-center"/>
 </element>
-<element name="C5" library="SparkFun-Capacitors" package="0603" value="22uF" x="9.271" y="4.318" smashed="yes" rot="R180">
+<element name="C4" library="SparkFun-Capacitors" package="0603" value="22uF" x="9.271" y="4.318" smashed="yes" rot="R180">
 <attribute name="NAME" x="9.271" y="3.556" size="0.6096" layer="25" font="vector" ratio="20" rot="R180" align="bottom-center"/>
 <attribute name="PROD_ID" value="CAP-14464" x="-30.099" y="15.748" size="1.778" layer="27" rot="R180" display="off"/>
@@
 <attribute name="VALUE" x="4.699" y="4.064" size="0.6096" layer="27" font="vector" ratio="20" align="bottom-center"/>
 </element>
-<element name="C2" library="SparkFun-Capacitors" package="0603" value="4.7uF" x="4.318" y="4.318" smashed="yes">
-<attribute name="NAME" x="4.318" y="5.08" size="0.6096" layer="25" font="vector" ratio="20" align="bottom-center"/>
-<attribute name="PROD_ID" value="CAP-14106" x="4.318" y="4.318" size="1.778" layer="27" font="vector" ratio="15" display="off"/>
-<attribute name="VALUE" x="4.318" y="3.556" size="0.6096" layer="27" font="vector" ratio="20" align="top-center"/>
-</element>
-<element name="C1" library="SparkFun-Capacitors" package="0603" value="4.7uF" x="4.318" y="2.794" smashed="yes">
-<attribute name="NAME" x="4.318" y="3.556" size="0.6096" layer="25" font="vector" ratio="20" align="bottom-center"/>
-<attribute name="PROD_ID" value="CAP-14106" x="4.318" y="2.794" size="1.778" layer="27" font="vector" ratio="15" display="off"/>
-<attribute name="VALUE" x="4.318" y="2.032" size="0.6096" layer="27" font="vector" ratio="20" align="top-center"/>
+<element name="C1" library="SparkFun-Capacitors" package="1210" value="10uF" x="4.953" y="3.683" smashed="yes">
+<attribute name="NAME" x="4.953" y="4.445" size="0.6096" layer="25" font="vector" ratio="20" align="bottom-center"/>
+<attribute name="PROD_ID" value="CAP-09824" x="4.953" y="3.683" size="1.778" layer="27" font="vector" ratio="15" display="off"/>
+<attribute name="VALUE" value="10uF" x="4.953" y="2.921" size="0.6096" layer="27" font="vector" ratio="20" align="top-center"/>
 </element>
 <element name="J1" library="SparkFun-Connectors" package="1X04_NO_SILK" value="" x="1.27" y="8.89" smashed="yes" rot="R270">
@@
 <element name="U$6" library="output" package="BREAKOUT0" value="" x="7.747" y="6.858" smashed="yes" rot="MR90"/>
 <element name="U$7" library="output" package="AP632030" value="" x="10.668" y="6.731" smashed="yes" rot="MR90"/>
+<element name="LOGO3" library="SparkFun-Aesthetics" package="ORDERING_INSTRUCTIONS" value="SPECIAL_INSTRUCTIONS-ORDERING" x="24.13" y="44.45" smashed="yes"/>
 </elements>
 <signals>
 <signal name="GND">
 <contactref element="U1" pad="4"/>
+<contactref element="C3" pad="2"/>
 <contactref element="C4" pad="2"/>
-<contactref element="C5" pad="2"/>
 <via x="4.699" y="5.461" extent="1-16" drill="0.3048"/>
-<via x="7.112" y="4.699" extent="1-16" drill="0.3048"/>
-<via x="7.112" y="3.556" extent="1-16" drill="0.3048"/>
-<via x="7.112" y="2.413" extent="1-16" drill="0.3048"/>
-<contactref element="C2" pad="2"/>
+<via x="5.461" y="4.572" extent="1-16" drill="0.3048"/>
+<via x="5.461" y="3.683" extent="1-16" drill="0.3048"/>
+<via x="5.461" y="2.667" extent="1-16" drill="0.3048"/>
 <polygon width="0.2032" layer="1" isolate="0.3048" thermals="no" rank="2">
-<vertex x="0" y="0"/>
-<vertex x="12.7" y="0"/>
-<vertex x="12.7" y="10.16"/>
-<vertex x="0" y="10.16"/>
+<vertex x="4.318" y="2.286"/>
+<vertex x="6.096" y="2.286"/>
+<vertex x="6.096" y="0.635"/>
+<vertex x="9.017" y="0.635"/>
+<vertex x="9.017" y="5.969"/>
+<vertex x="4.318" y="5.969"/>
 </polygon>
 <polygon width="0.2032" layer="16" isolate="0.3048" thermals="no" rank="2">
@@
 <signal name="N$4">
 <contactref element="U1" pad="6"/>
-<contactref element="C3" pad="1"/>
+<contactref element="C2" pad="1"/>
 <wire x1="6.0741" y1="7.554" x2="5.273" y2="7.554" width="0.2032" layer="1"/>
 <wire x1="5.273" y1="7.554" x2="4.992" y2="7.835" width="0.2032" layer="1"/>
@@
 <contactref element="U1" pad="5"/>
 <contactref element="L1" pad="P$1"/>
-<contactref element="C3" pad="2"/>
+<contactref element="C2" pad="2"/>
 <polygon width="0.2032" layer="1" isolate="0.3048" thermals="no">
-<vertex x="5.461" y="6.35"/>
+<vertex x="5.334" y="6.35"/>
 <vertex x="7.62" y="6.35"/>
 <vertex x="7.62" y="5.334"/>
 <vertex x="9.017" y="5.334"/>
 <vertex x="9.017" y="9.525"/>
-<vertex x="6.223" y="9.525"/>
-<vertex x="6.223" y="8.509"/>
+<vertex x="6.096" y="9.525"/>
+<vertex x="6.096" y="8.509"/>
 <vertex x="7.239" y="8.509"/>
 <vertex x="7.239" y="6.858"/>
-<vertex x="5.461" y="6.858"/>
+<vertex x="5.334" y="6.858"/>
 </polygon>
 </signal>
@@
 <contactref element="U1" pad="3"/>
 <contactref element="C1" pad="1"/>
-<contactref element="C2" pad="1"/>
 <contactref element="R1" pad="2"/>
 <polygon width="0.2032" layer="1" isolate="0.3048" thermals="no">
@@
 <signal name="3.3V">
 <contactref element="L1" pad="P$2"/>
-<contactref element="C5" pad="1"/>
 <contactref element="C4" pad="1"/>
+<contactref element="C3" pad="1"/>
 <contactref element="U1" pad="1"/>
 <polygon width="0.2032" layer="1" isolate="0.3048" thermals="no">
@@
 <vertex x="9.652" y="0"/>
 <vertex x="9.652" y="5.969"/>
-<vertex x="8.509" y="7.112"/>
-<vertex x="0" y="7.112"/>
+<vertex x="7.747" y="7.874"/>
+<vertex x="0" y="7.874"/>
 </polygon>
 <polygon width="0.2032" layer="1" isolate="0.3048" thermals="no">
 <vertex x="0" y="10.16"/>
-<vertex x="5.08" y="10.16"/>
-<vertex x="5.08" y="7.366"/>
-<vertex x="0" y="7.366"/>
+<vertex x="4.064" y="10.16"/>
+<vertex x="4.064" y="7.239"/>
+<vertex x="0" y="7.239"/>
 </polygon>
 <via x="10.16" y="8.89" extent="1-16" drill="0.3048"/>
@@
 </signals>
 <mfgpreviewcolors>
-<mfgpreviewcolor name="soldermaskcolor" color="0xC8008000"/>
+<mfgpreviewcolor name="soldermaskcolor" color="0xC8DC1518"/>
 <mfgpreviewcolor name="silkscreencolor" color="0xFFFEFEFE"/>
 <mfgpreviewcolor name="backgroundcolor" color="0xFF282828"/>

Commit message: Update SparkFun Buck Regulator Breakout - AP63203.brd
Parts:
- removed U$5: (no value), output:BUCK0
- added U$8: (no value), output:BABYBUCK0
- moved U$6 0.13 mm to (7.75, 6.73)
Changed lines of the file:
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@@
 <layer number="27" name="tValues" color="7" fill="1" visible="no" active="yes"/>
 <layer number="28" name="bValues" color="7" fill="1" visible="no" active="yes"/>
-<layer number="29" name="tStop" color="7" fill="3" visible="yes" active="yes"/>
+<layer number="29" name="tStop" color="7" fill="3" visible="no" active="yes"/>
 <layer number="30" name="bStop" color="7" fill="6" visible="no" active="yes"/>
 <layer number="31" name="tCream" color="7" fill="4" visible="no" active="yes"/>
@@
 <layer number="37" name="tTest" color="7" fill="1" visible="no" active="yes"/>
 <layer number="38" name="bTest" color="7" fill="1" visible="no" active="yes"/>
-<layer number="39" name="tKeepout" color="4" fill="11" visible="yes" active="yes"/>
-<layer number="40" name="bKeepout" color="1" fill="11" visible="yes" active="yes"/>
+<layer number="39" name="tKeepout" color="4" fill="11" visible="no" active="yes"/>
+<layer number="40" name="bKeepout" color="1" fill="11" visible="no" active="yes"/>
 <layer number="41" name="tRestrict" color="4" fill="10" visible="no" active="yes"/>
 <layer number="42" name="bRestrict" color="1" fill="10" visible="no" active="yes"/>
@@
 <layer number="50" name="dxf" color="7" fill="1" visible="no" active="no"/>
 <layer number="51" name="tDocu" color="6" fill="1" visible="yes" active="yes"/>
-<layer number="52" name="bDocu" color="7" fill="1" visible="no" active="yes"/>
+<layer number="52" name="bDocu" color="7" fill="1" visible="yes" active="yes"/>
 <layer number="53" name="tGND_GNDA" color="7" fill="9" visible="no" active="no"/>
 <layer number="54" name="bGND_GNDA" color="1" fill="9" visible="no" active="no"/>
@@
 <element name="LOGO1" library="SparkFun-Aesthetics" package="SFE_LOGO_FLAME_.1" value="SFE_LOGO_FLAME.1_INCH" x="8.128" y="1.524" smashed="yes" rot="MR90"/>
 <element name="LOGO2" library="SparkFun-Aesthetics" package="OSHW-LOGO-S" value="OSHW-LOGOS" x="10.795" y="1.905" smashed="yes" rot="MR90"/>
-<element name="U$5" library="output" package="BUCK0" value="" x="9.271" y="5.334" smashed="yes" rot="MR90"/>
-<element name="U$6" library="output" package="BREAKOUT0" value="" x="7.747" y="6.858" smashed="yes" rot="MR90"/>
+<element name="U$6" library="output" package="BREAKOUT0" value="" x="7.747" y="6.731" smashed="yes" rot="MR90"/>
 <element name="U$7" library="output" package="AP632030" value="" x="10.668" y="6.731" smashed="yes" rot="MR90"/>
 <element name="LOGO3" library="SparkFun-Aesthetics" package="ORDERING_INSTRUCTIONS" value="SPECIAL_INSTRUCTIONS-ORDERING" x="24.13" y="44.45" smashed="yes"/>
+<element name="U$8" library="output" package="BABYBUCK0" value="" x="9.271" y="3.175" smashed="yes" rot="MR90"/>
 </elements>
 <signals>
