File: SparkFun BabyBuck Regulator - AP63203/Hardware/SparkFun BabyBuck Regulator - AP63203.brd (EAGLE design)
At the start: 12.7 x 10.2 mm, 24 parts, among them U1 AP63203

Commit message: V10
Parts:
- removed U$6: (no value), output:BREAKOUT0
- moved U$8 5.22 mm to (12.7, 7.11), turned to 0 degrees
- moved U$7 1.83 mm to (9.14, 5.71), turned to 0 degrees
- moved LOGO1 1.57 mm to (7.75, 3.05), turned to 0 degrees
- moved LOGO2 1.15 mm to (10.7, 3.05), turned to 0 degrees
Other:
- board text added: "V10"
- board text removed: "v01"
Changed lines of the file:
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@@
 <layer number="50" name="dxf" color="7" fill="1" visible="no" active="no"/>
 <layer number="51" name="tDocu" color="6" fill="1" visible="yes" active="yes"/>
-<layer number="52" name="bDocu" color="7" fill="1" visible="yes" active="yes"/>
+<layer number="52" name="bDocu" color="7" fill="1" visible="no" active="yes"/>
 <layer number="53" name="tGND_GNDA" color="7" fill="9" visible="no" active="no"/>
 <layer number="54" name="bGND_GNDA" color="1" fill="9" visible="no" active="no"/>
@@
 <dimension x1="0" y1="0" x2="0" y2="10.16" x3="-2.54" y3="5.08" textsize="1.27" textratio="15" layer="47" unit="inch"/>
 <text x="10.16" y="-15.24" size="1.778" layer="51" font="vector" ratio="15">Alex Wende</text>
-<text x="12.192" y="9.779" size="1.016" layer="16" font="vector" ratio="15" rot="SMR270">v01</text>
+<text x="9.906" y="9.779" size="1.016" layer="16" font="vector" ratio="15" rot="SMR180">V10</text>
 <text x="25.4" y="31.75" size="1.778" layer="51" font="vector" ratio="15">2oz copper</text>
 </plain>
@@
 <element name="U$4" library="output" package="#EN#0" value="" x="3.429" y="1.27" smashed="yes" rot="MR0"/>
 <element name="U$3" library="output" package="#VIN#0" value="" x="3.556" y="3.81" smashed="yes" rot="MR0"/>
-<element name="LOGO1" library="SparkFun-Aesthetics" package="SFE_LOGO_FLAME_.1" value="SFE_LOGO_FLAME.1_INCH" x="8.128" y="1.524" smashed="yes" rot="MR90"/>
-<element name="LOGO2" library="SparkFun-Aesthetics" package="OSHW-LOGO-S" value="OSHW-LOGOS" x="10.795" y="1.905" smashed="yes" rot="MR90"/>
-<element name="U$6" library="output" package="BREAKOUT0" value="" x="7.747" y="6.731" smashed="yes" rot="MR90"/>
-<element name="U$7" library="output" package="AP632030" value="" x="10.668" y="6.731" smashed="yes" rot="MR90"/>
+<element name="LOGO1" library="SparkFun-Aesthetics" package="SFE_LOGO_FLAME_.1" value="SFE_LOGO_FLAME.1_INCH" x="7.747" y="3.048" smashed="yes" rot="MR0"/>
+<element name="LOGO2" library="SparkFun-Aesthetics" package="OSHW-LOGO-S" value="OSHW-LOGOS" x="10.668" y="3.048" smashed="yes" rot="MR0"/>
+<element name="U$7" library="output" package="AP632030" value="" x="9.144" y="5.715" smashed="yes" rot="MR0"/>
 <element name="LOGO3" library="SparkFun-Aesthetics" package="ORDERING_INSTRUCTIONS" value="SPECIAL_INSTRUCTIONS-ORDERING" x="24.13" y="44.45" smashed="yes"/>
-<element name="U$8" library="output" package="BABYBUCK0" value="" x="9.271" y="3.175" smashed="yes" rot="MR90"/>
+<element name="U$8" library="output" package="BABYBUCK0" value="" x="12.7" y="7.112" smashed="yes" rot="MR0"/>
 </elements>
 <signals>
@@
 <vertex x="0" y="7.239"/>
 </polygon>
-<via x="10.16" y="8.89" extent="1-16" drill="0.3048"/>
+<via x="10.16" y="8.382" extent="1-16" drill="0.3048"/>
 </signal>
 <signal name="EN">
