File: SparkFun Buck Regulator - AP63203/Hardware/Production/SparkFun Buck Regulator - AP63203-Panel.brd (EAGLE design)
At the start: 149.1 x 200.9 mm, 1511 parts, among them J102 POWER_JACK, J105 POWER_JACK, J12 POWER_JACK, J15 POWER_JACK, J18 POWER_JACK, J21 POWER_JACK, J24 POWER_JACK, J27 POWER_JACK, J3 POWER_JACK, J30 POWER_JACK, J33 POWER_JACK, J36 POWER_JACK, J39 POWER_JACK, J42 POWER_JACK, J45 POWER_JACK, J48 POWER_JACK, J51 POWER_JACK, J54 POWER_JACK, J57 POWER_JACK, J6 POWER_JACK, J60 POWER_JACK, J63 POWER_JACK, J66 POWER_JACK, J69 POWER_JACK, J72 POWER_JACK, J75 POWER_JACK, J78 POWER_JACK, J81 POWER_JACK, J84 POWER_JACK, J87 POWER_JACK, J9 POWER_JACK, J90 POWER_JACK, J93 POWER_JACK, J96 POWER_JACK, J99 POWER_JACK, U1 AP63203, U10 AP63203, U11 AP63203, U12 AP63203, U13 AP63203, U14 AP63203, U15 AP63203, U16 AP63203, U17 AP63203, U18 AP63203, U19 AP63203, U2 AP63203, U20 AP63203, U21 AP63203, U22 AP63203, U23 AP63203, U24 AP63203, U25 AP63203, U26 AP63203, U27 AP63203, U28 AP63203, U29 AP63203, U3 AP63203, U30 AP63203, U31 AP63203, U32 AP63203, U33 AP63203, U34 AP63203, U35 AP63203, U4 AP63203, U5 AP63203, U6 AP63203, U7 AP63203, U8 AP63203, U9 AP63203

Commit message: Updated barrel jack silk
Parts:
- moved E$1 1.59 mm to (-2.62, 178.2)
- moved E$2 1.59 mm to (-2.62, 178.2)
- moved E$3 1.59 mm to (131.7, 178.2)
- moved E$4 1.59 mm to (131.7, 178.2)
- moved E$5 0.51 mm to (-2.62, 6.35)
- moved E$6 0.51 mm to (-2.62, 6.35)
Other:
- board size 149.1 x 200.9 mm -> 149.1 x 195.1 mm
